File: clockport nic.brd (EAGLE design)
At the start: 40 x 70 mm, 54 parts, among them CN1 J1011F21P, CN2 MOLEX-MILLIGRID-22W-87758-2216, Q1 3904, Q2 3904, U1 KSZ8851-16MLL, U2 74LVC02PW, U3 74LVC245PW, U4 74LVC00PW, U5 1117MPX-3.3

Commit message: Add files via upload
Parts:
- removed Q1, Q2: 3904, jc-discretesemi:SOT23
- removed R12: 4K7, rcl:R0603
- added U6: 74LVC1G07DBV, jc-logic:SOT23-5
- D2: value 1N4148W -> BAS16; device jc-discretesemi:SOD-123 -> jc-discretesemi:SOD323-R
- R11: value 4K7 -> 1K
- R8: value 1K -> 4K7
- moved R8 6.02 mm to (32.1, 19.8)
- moved R11 4.83 mm to (32.1, 23.6)
- moved L1 1.65 mm to (10.8, 23.9)
- moved C18 1.40 mm to (31.9, 31.5)
- moved U5 1.27 mm to (7.62, 35.6)
- moved C14 1.27 mm to (4.06, 30.5)
- moved D2 1.27 mm to (31.1, 14.6)
- moved L2 1.27 mm to (10.8, 29.5)
- moved R9 1.27 mm to (32.1, 17.9)
- moved TP1 1.27 mm to (19.1, 11.4)
- moved TP2 1.27 mm to (17.1, 11.4)
- moved TP3 1.27 mm to (20.3, 19.1)
- moved C15 1.27 mm to (7.87, 41.3)
- moved R10 0.76 mm to (32.1, 21.7)
- moved TP4 0.64 mm to (24.8, 17.8)
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Connections:
- removed net N$3: Q1.1, Q2.3, R11.1
- net !INT6: now also U6.4; no longer Q1.3
- net !KS_INT: now also R8.1, U6.2; no longer Q2.1, R10.1
- net +3V3D: now also R8.2, U6.5; no longer R11.2, R12.2
- net EEPROM_SCK: now also R10.1; no longer R12.1
- net GND1: now also R11.2, U6.3; no longer Q1.2, Q2.2, R8.2
- net LED1: now also R11.1; no longer R8.1
Routing:
- net N$3: track 12.0 -> 0.00 mm
- net !KS_INT: track 22.9 -> 17.6 mm, vias 2 -> 1
- net !INT6: track 27.9 -> 31.8 mm
- net GND1: track 24.6 -> 27.9 mm, vias 133 -> 142
- net +3V3D: track 99.4 -> 96.2 mm
- net EEPROM_SCK: track 12.6 -> 15.3 mm
- net !KS_RST: track 24.1 -> 21.8 mm
- net !RESET: track 7.04 -> 8.81 mm
- net KS_A/!D: track 29.7 -> 28.0 mm
- net N$8: track 11.6 -> 13.0 mm
- net !KS_WR: track 27.9 -> 26.5 mm
- net !KS_RD: track 26.8 -> 25.5 mm
- net 3V3A: track 44.8 -> 43.6 mm, vias 4 -> 3
- net !KS_CS: track 24.5 -> 23.3 mm
- net +5V: track 30.2 -> 31.4 mm
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Other:
- board text removed: "Plug in baby!"
