File: clockport nic.sch (EAGLE design)
At the start: 54 parts, among them CN1 J1011F21P, CN2 MOLEX-MILLIGRID-22W-87758-2216, Q1 3904, Q2 3904, U1 KSZ8851-16MLL, U2 74LVC02PW, U3 74LVC245PW, U4 74LVC00PW, U5 1117MPX-3.3

Commit message: Add files via upload
Parts:
- removed Q1, Q2: 3904, jc-discretesemi:-NPN_SOT23
- removed R12: 4K7, rcl:R-EU_R0603
- added U6: 74LVC1G07DBV, jc-logic:74LVC1G07DBV
- D2: value 1N4148W -> BAS16; device jc-discretesemi:-DIODE_SOD-123 -> jc-discretesemi:-DIODE_SOD-323
- R11: value 4K7 -> 1K
- R8: value 1K -> 4K7
Connections:
- removed net N$3: Q1.B, Q2.C, R11.1
- net !INT6: now also U6A.O; no longer Q1.C
- net !KS_INT: now also R8.1, U6A.I; no longer Q2.B, R10.1
- net +3V3D: now also R8.2, U6P.VCC; no longer R11.2, R12.2
- net EEPROM_SCK: now also R10.1; no longer R12.1
- net GND1: now also R11.2, U6P.GND; no longer Q1.E, Q2.E, R8.2
- net LED1: now also R11.1; no longer R8.1
